File: HW/GroundRobot/GroundRobot.kicad_sch (KiCad schematic)
At the start: 1 part, among them U1 ESP32

Commit message: update pcb and latex
Parts:
- removed U1: ESP32, Package_DFN_QFN:QFN-48-1EP_6x6mm_P0.4mm_EP4.3x4.3mm, symbol Espressif:ESP32
- added U1: ESP32, Module:Arduino_UNO_R3_WithMountingHoles, symbol Espressif:ESP32-WEMOS-D1-R32
Connections:
- new net: U1.1 (VDDA), U1.43 (VDDA), U1.46 (VDDA)
- new net: U1.3 (VDD3P3), U1.4 (VDD3P3)
- new net Motor Drivers/Pitch Direction: U1.34 (GPIO5)
- new net Motor Drivers/Pitch Step: U1.20 (MTCK/GPIO13/ADC2_CH4)
- new net Motor Drivers/Roll Direction: U1.18 (MTDI/GPIO12/ADC2_CH5)
- new net Motor Drivers/Roll Step: U1.17 (MTMS/GPIO14/ADC2_CH6)
Other:
- added sheet Motor Drivers (MotoDrivers.kicad_sch)
- company: (none) -> Emerson Kazuyoshi Kaneda
- title: (none) -> Self-Stabilize Shield Module
Changed lines of the file:
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@@
 (kicad_sch (version 20230121) (generator eeschema)
   (paper "A4")
-  (symbol (lib_id "Espressif:ESP32") (at 147.32 97.79 0) (unit 1)
+  (title_block
+    (title "Self-Stabilize Shield Module")
+    (date "2024-08-06")
+    (rev "1.0")
+    (company "Emerson Kazuyoshi Kaneda")
+    (comment 1 "Universidade Tecnológica Federal do Paraná (UTFPR)")
+    (comment 2 "Instituto Politécnico de Bragança (IPB)")
+    (comment 3 "Centro de Digitalização de Robótica Inteligente (CeDRI)")
+  )
+  (wire (pts (xy 99.06 90.17) (xy 111.76 90.17))
+    (stroke (width 0) (type default))
+  )
+  (wire (pts (xy 96.52 97.79) (xy 96.52 85.09))
+    (stroke (width 0) (type default))
+  )
+  (wire (pts (xy 92.71 85.09) (xy 92.71 38.1))
+    (stroke (width 0) (type default))
+  )
+  (wire (pts (xy 76.2 100.33) (xy 99.06 100.33))
+    (stroke (width 0) (type default))
+  )
+  (wire (pts (xy 96.52 85.09) (xy 111.76 85.09))
+    (stroke (width 0) (type default))
+  )
+  (wire (pts (xy 92.71 38.1) (xy 193.04 38.1))
+    (stroke (width 0) (type default))
+  )
+  (wire (pts (xy 76.2 97.79) (xy 96.52 97.79))
+    (stroke (width 0) (type default))
+  )
+  (wire (pts (xy 76.2 85.09) (xy 92.71 85.09))
+    (stroke (width 0) (type default))
+  )
+  (wire (pts (xy 177.8 77.47) (xy 193.04 77.47))
+    (stroke (width 0) (type default))
+  )
+  (wire (pts (xy 76.2 87.63) (xy 111.76 87.63))
+    (stroke (width 0) (type default))
+  )
+  (wire (pts (xy 193.04 38.1) (xy 193.04 77.47))
+    (stroke (width 0) (type default))
+  )
+  (wire (pts (xy 99.06 100.33) (xy 99.06 90.17))
+    (stroke (width 0) (type default))
+  )
+  (symbol (lib_id "Espressif:ESP32-WEMOS-D1-R32") (at 144.78 92.71 0) (unit 1)
     (in_bom yes) (on_board yes) (dnp no) (fields_autoplaced)
-    (property "Reference" "U1" (at 149.2759 135.89 0)
+    (property "Reference" "U1" (at 146.7359 130.81 0)
       (effects (font (size 1.27 1.27)) (justify left))
     )
-    (property "Value" "ESP32" (at 149.2759 138.43 0)
+    (property "Value" "ESP32" (at 146.7359 133.35 0)
       (effects (font (size 1.27 1.27)) (justify left))
     )
-    (property "Footprint" "Package_DFN_QFN:QFN-48-1EP_6x6mm_P0.4mm_EP4.3x4.3mm" (at 147.32 146.05 0)
+    (property "Footprint" "Module:Arduino_UNO_R3_WithMountingHoles" (at 144.78 140.97 0)
       (effects (font (size 1.27 1.27)) hide)
     )
-    (property "Datasheet" "https://www.espressif.com/sites/default/files/documentation/esp32_datasheet_en.pdf" (at 147.32 148.59 0)
+    (property "Datasheet" "https://www.espressif.com/sites/default/files/documentation/esp32_datasheet_en.pdf" (at 144.78 143.51 0)
       (effects (font (size 1.27 1.27)) hide)
     )
@@
       )
     )
+  )
+  (sheet (at 36.83 74.93) (size 39.37 34.29) (fields_autoplaced)
+    (stroke (width 0.1524) (type solid))
+    (fill (color 0 0 0 0.0000))
+    (property "Sheetname" "Motor Drivers" (at 36.83 74.2184 0)
+      (effects (font (size 1.27 1.27)) (justify left bottom))
+    )
+    (property "Sheetfile" "MotoDrivers.kicad_sch" (at 36.83 109.8046 0)
+      (effects (font (size 1.27 1.27)) (justify left top) hide)
+    )
+    (pin "Pitch Direction" input (at 76.2 85.09 0)
+      (effects (font (size 1.27 1.27)) (justify right))
+    )
+    (pin "Roll Direction" input (at 76.2 97.79 0)
+      (effects (font (size 1.27 1.27)) (justify right))
+    )
+    (pin "VMOT" input (at 64.77 74.93 90)
+      (effects (font (size 1.27 1.27)) (justify right))
+    )
+    (pin "+5V" input (at 50.8 74.93 90)
+      (effects (font (size 1.27 1.27)) (justify right))
+    )
+    (pin "Roll Step" input (at 76.2 100.33 0)
+      (effects (font (size 1.27 1.27)) (justify right))
+    )
+    (pin "GND" input (at 58.42 109.22 270)
+      (effects (font (size 1.27 1.27)) (justify left))
+    )
+    (pin "Pitch Step" input (at 76.2 87.63 0)
+      (effects (font (size 1.27 1.27)) (justify right))
+    )
+    (instances
+      (project "GroundRobot"
+        (path "/566a287a-263c-4e32-9545-a9a2397aa7b1" (page "2"))
+      )
+    )

Commit message: update HW and tests
Parts:
- added A1: Pitch, Module:Pololu_Breakout-16_15.2x20.3mm, symbol Driver_Motor:Pololu_Breakout_DRV8825
- added A2: Roll, Module:Pololu_Breakout-16_15.2x20.3mm, symbol Driver_Motor:Pololu_Breakout_DRV8825
- added AE1: Antenna, symbol Device:Antenna
- added BT1: Battery, symbol Device:Battery
- added M1, M2: NEMA17, symbol Motor:Stepper_Motor_bipolar
- added R1, R2, R3, R4, R5, R6, R7, R8: 10k, symbol Device:R
- added SW1: SW_SPST, symbol Switch:SW_SPST
- added U2: LM2596S-ADJ, Package_TO_SOT_SMD:TO-263-5_TabPin3, symbol Regulator_Switching:LM2596S-ADJ
- added U3: ADXL343, Package_LGA:LGA-14_3x5mm_P0.8mm_LayoutBorder1x6y, symbol Sensor_Motion:ADXL343
- added U4: ~, symbol Interfaces:HC-12
Connections:
- net +5V: now reaches U1.1 (VDDA), U1.43 (VDDA), U1.46 (VDDA)
- net +5V: now also A1.13 (~{RST}), A1.14 (~{SLP}), A1.2 (~{FLT}), A2.13 (~{RST}), A2.14 (~{SLP}), A2.2 (~{FLT}), R1.1, R2.1, R3.1, R4.1, R5.1, R6.1, R7.2, R8.2, U2.2 (OUT), U3.6 (Vs), U4.1 (VCC)
- net SCL: now reaches U1.39 (GPIO22)
- net SCL: now also R7.1, U3.14 (SCL/SCLK)
- net RX: now reaches U1.40 (U0RXD/GPIO3)
- net RX: now also U4.4 (TXD)
- net TX: now reaches U1.41 (U0TXD/GPIO1)
- net TX: now also U4.3 (RXD)
- net SDA: now reaches U1.42 (GPIO21)
- net SDA: now also R8.1, U3.13 (SDA/SDI/SDIO)
- net GND: now reaches U1.49 (GND)
- net GND: now also A1.1 (GND), A1.7 (GND), A2.1 (GND), A2.7 (GND), BT1.2 (-), U2.3 (GND), U3.2 (GND), U3.4 (GND), U3.5 (GND), U4.2 (GND)
- net Motor Drivers/Pitch Direction renamed Pitch_dir
- net Pitch_dir: now also A1.16 (DIR)
- net Motor Drivers/Pitch Step renamed Pitch_step
- net Pitch_step: now also A1.15 (STEP)
- net Motor Drivers/Roll Direction renamed Roll_dir
- net Roll_dir: now also A2.16 (DIR)
- net Motor Drivers/Roll Step renamed Roll_step
- net Roll_step: now also A2.15 (STEP)
- new net: A2.3 (A2), M2.1
- new net: A2.4 (A1), M2.2 (-)
- new net: A2.5 (B1), M2.3
- new net: A2.6 (B2), M2.4
- new net: A2.10 (M0), R4.2
- new net: AE1.1 (A), U4. (GND@8)
- new net: A1.12 (M2), R3.2
- new net: A1.3 (A2), M1.1
- new net: A1.4 (A1), M1.2 (-)
- new net: A1.5 (B1), M1.3
- new net: A1.6 (B2), M1.4
- new net: A2.12 (M2), R6.2
- new net: A1.10 (M0), R1.2
- new net: A1.11 (M1), R2.2
- new net: A2.11 (M1), R5.2
- new net: BT1.1 (+), SW1.1 (A)
- new net +12V: A1.8 (VMOT), A2.8 (VMOT), SW1.2 (B), U2.1 (VIN)
Other:
- removed sheet Motor Drivers
- moved on the sheet: U1
